Commit message: 2 robot launch testing continued

File: two_robot_sim/urdf/robot1.urdf (robot description, URDF)
Before this commit: robot robot1, 5 links, 4 joints
Links:
- added link dummy_root
- link camera_link: mass 0.1 -> 0.2
- link lidar_link: mass 0.1 -> 0.3
Joints:
- added joint dummy_joint: type fixed, parent dummy_root, child base_link
- joint camera_joint: origin xyz=0.2 0 0.1 rpy=0 0 0 -> xyz=0.2 0 0.15 rpy=0 0 0
- joint left_wheel_joint: origin xyz=-0.2 0.25 -0.05 rpy=0 0 0 -> xyz=-0.2 0.25 0.05 rpy=0 0 0
- joint lidar_joint: origin xyz=0.2 0 0.2 rpy=0 0 0 -> xyz=0.2 0 0.25 rpy=0 0 0
- joint right_wheel_joint: origin xyz=-0.2 -0.25 -0.05 rpy=0 0 0 -> xyz=-0.2 -0.25 0.05 rpy=0 0 0

File: two_robot_sim/urdf/robot2.urdf (robot description, URDF)
Before this commit: robot robot2, 5 links, 4 joints
Links:
- added link dummy_root
- link camera_link: mass 0.1 -> 0.2
- link lidar_link: mass 0.1 -> 0.3
Joints:
- added joint dummy_joint: type fixed, parent dummy_root, child base_link
- joint camera_joint: origin xyz=0.2 0 0.1 rpy=0 0 0 -> xyz=0.2 0 0.15 rpy=0 0 0
- joint left_wheel_joint: origin xyz=-0.2 0.25 -0.05 rpy=0 0 0 -> xyz=-0.2 0.25 0.05 rpy=0 0 0
- joint lidar_joint: origin xyz=0.2 0 0.2 rpy=0 0 0 -> xyz=0.2 0 0.25 rpy=0 0 0
- joint right_wheel_joint: origin xyz=-0.2 -0.25 -0.05 rpy=0 0 0 -> xyz=-0.2 -0.25 0.05 rpy=0 0 0

Commit message: lidar and diff crive yet to complete

File: two_robot_sim/urdf/robot1.urdf (robot description, URDF)
Before this commit: robot robot1, 6 links, 5 joints
Links:
- added link caster_wheel, mass 1; collision sphere radius=0.03; visual sphere radius=0.03
- link camera_link: geometry collision box size=0.025 0.025 0.025; visual box size=0.025 0.025 0.025
Joints:
- added joint caster_joint: type fixed, parent base_link, child caster_wheel, origin xyz=0.15 0 -0.03 rpy=0 0 0
- joint camera_joint: origin xyz=0.2 0 0.15 rpy=0 0 0 -> xyz=0.2 0 0.05 rpy=0 0 0
- joint left_wheel_joint: origin xyz=-0.2 0.25 0.05 rpy=0 0 0 -> xyz=-0.15 0.225 0.05 rpy=0 0 0
- joint lidar_joint: origin xyz=0.2 0 0.25 rpy=0 0 0 -> xyz=0.0 0 0.15 rpy=0 0 0
- joint right_wheel_joint: origin xyz=-0.2 -0.25 0.05 rpy=0 0 0 -> xyz=-0.15 -0.225 0.05 rpy=0 0 0

File: two_robot_sim/urdf/robot2.urdf (robot description, URDF)
Before this commit: robot robot2, 6 links, 5 joints
Links:
- added link caster_wheel, mass 1; collision sphere radius=0.03; visual sphere radius=0.03
- link camera_link: geometry collision box size=0.025 0.025 0.025; visual box size=0.025 0.025 0.025
Joints:
- added joint caster_joint: type fixed, parent base_link, child caster_wheel, origin xyz=0.15 0 -0.03 rpy=0 0 0
- joint camera_joint: origin xyz=0.2 0 0.15 rpy=0 0 0 -> xyz=0.2 0 0.05 rpy=0 0 0
- joint left_wheel_joint: origin xyz=-0.2 0.25 0.05 rpy=0 0 0 -> xyz=-0.15 0.225 0.05 rpy=0 0 0
- joint lidar_joint: origin xyz=0.2 0 0.25 rpy=0 0 0 -> xyz=0.0 0 0.15 rpy=0 0 0
- joint right_wheel_joint: origin xyz=-0.2 -0.25 0.05 rpy=0 0 0 -> xyz=-0.15 -0.225 0.05 rpy=0 0 0
